File: hw/fpga.sch (KiCad schematic (older format))
At the start: 60 parts, among them P10 CONN_01X01, P11 CONN_01X01, P12 CONN_01X01, P13 CONN_01X01, P14 CONN_01X01, P15 CONN_01X01, P16 CONN_01X01, P26 TP, P27 TP, P28 CONN_01X01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

Commit message: Update components values
Change IF amplifier to ADA4940. Same footprint, no changes in PCB.
Fix M[0:2] connections.
Parts:
- R110: value 1k -> DNP
- R115: value 0 -> DNP
- R116: value DNP -> 0
- SW1: value SW_PUSH -> DNP
Changed lines of the file:
@@
 P 750 7150
 F 0 "SW1" H 900 7260 50  0000 C CNN
-F 1 "SW_PUSH" H 750 7070 50  0000 C CNN
+F 1 "DNP" H 750 7070 50  0000 C CNN
 F 2 "VNA:EVP-AWBA2A" H 750 7150 60  0001 C CNN
 F 3 "" H 750 7150 60  0000 C CNN
@@
 P 1450 7100
 F 0 "R115" V 1530 7100 50  0000 C CNN
-F 1 "0" V 1450 7100 50  0000 C CNN
+F 1 "DNP" V 1450 7100 50  0000 C CNN
 F 2 "VNA:R_0402b" V 1380 7100 30  0001 C CNN
 F 3 "" H 1450 7100 30  0000 C CNN
@@
 P 1450 7500
 F 0 "R116" V 1530 7500 50  0000 C CNN
-F 1 "DNP" V 1450 7500 50  0000 C CNN
+F 1 "0" V 1450 7500 50  0000 C CNN
 F 2 "VNA:R_0402b" V 1380 7500 30  0001 C CNN
 F 3 "" H 1450 7500 30  0000 C CNN
@@
 P 750 7800
 F 0 "R110" V 830 7800 50  0000 C CNN
-F 1 "1k" V 750 7800 50  0000 C CNN
+F 1 "DNP" V 750 7800 50  0000 C CNN
 F 2 "VNA:R_0402b" V 680 7800 30  0001 C CNN
 F 3 "" H 750 7800 30  0000 C CNN
