File: hw/if_amp.sch (KiCad schematic (older format))
At the start: 34 parts, among them U21 ADA4932-1

Commit message: Update components values
Change IF amplifier to ADA4940. Same footprint, no changes in PCB.
Fix M[0:2] connections.
Parts:
- U21: value ADA4932-1 -> ADA4940-1
Changed lines of the file:
@@
 P 6300 3900
 F 0 "U21" H 6300 3850 60  0000 C CNN
-F 1 "ADA4932-1" H 6850 4500 60  0000 C CNN
+F 1 "ADA4940-1" H 6850 4500 60  0000 C CNN
 F 2 "VNA:VFQFN-16" H 6100 3500 60  0001 C CNN
 F 3 "" H 6100 3500 60  0001 C CNN
